File: LoadCell-Main.sch (KiCad schematic (older format))
At the start: 47 parts, among them J1 M20-8760242, J2 0.100_1X4, J3 M20-8760242, J4 0.100_1X4, J5 M20-8760242, J6 0.100_1X4, J7 M20-8760242, J8 0.100_1X4, U3 L78L12ABUTR, U4 LM321SN3T1G, U5 L78L12ABUTR, U6 LM321SN3T1G, U7 L78L12ABUTR, U8 LM321SN3T1G

Commit message: Checkpoint
Parts:
- removed C4: 1uF, _Passive:C_0402, symbol C
- removed D2: MM3Z3V0ST1G, _Passive:SOD-323, symbol D_ZENER
- removed J3, J7: M20-8760242, _Connector:Pin_Header_Straight_2x02_Pitch2.54mm_SMD, symbol CONN_02X02
- removed J4, J6: 0.100_1X4, _Connector:0.100_1x4_micro, symbol 0.100_1X4
- removed R7, R8: 100R, _Passive:R_0402, symbol R
- removed U3, U5, U7: L78L12ABUTR, _Active:SOT89-3, symbol L78L12ABUTR
- removed U4, U6, U8: LM321SN3T1G, _Active:SOT-23-5, symbol LM321_23-5
- added C1, C10, C11, C12, C13, C14, C15, C16, C9: 1uF, _Passive:C_0603, symbol C
- added D1, D5, D6, D7, D8: MM3Z3V0ST1G, _Passive:SOD-323, symbol D_ZENER
- added J1, J10, J13, J14, J6, J9: M20-8760242, _Connector:Pin_Header_Straight_2x02_Pitch2.54mm_SMD, symbol CONN_02X02
- added J11, J12, J15, J16, J3, J7: 0.100_1X4, _Connector:0.100_1x4_micro, symbol 0.100_1X4
- added R1, R17, R19, R25, R27: 390K, _Passive:R_0603, symbol R
- added R18, R2, R20, R21, R23, R26, R28, R29, R31: 1K, _Passive:R_0603, symbol R
- added R22, R24, R30, R32: 270K, _Passive:R_0603, symbol R
- added U1, U3, U4, U5, U6, U7, U8: MCP6002, Housings_SSOP:TSSOP-8_4.4x3mm_Pitch0.65mm, symbol MCP6002
- C3, C5, C6, C7, C8: footprint _Passive:C_0402 -> _Passive:C_0603
- R10: footprint _Passive:R_0402 -> _Passive:R_0603
- R11: value 100R -> 390K; footprint _Passive:R_0402 -> _Passive:R_0603
- R12, R15: value 100R -> 1K; footprint _Passive:R_0402 -> _Passive:R_0603
- R13, R5: value 270K -> 1K; footprint _Passive:R_0402 -> _Passive:R_0603
- R14, R6: value 1K -> 270K; footprint _Passive:R_0402 -> _Passive:R_0603
- R16: value 100R -> 270K; footprint _Passive:R_0402 -> _Passive:R_0603
- R9: value 270K -> 390K; footprint _Passive:R_0402 -> _Passive:R_0603
- U2: renamed from U?; footprint (none) -> Housings_SSOP:TSSOP-8_4.4x3mm_Pitch0.65mm
- gave numbers to parts that had none: 2
- renumbered C1 to C4, D1 to D2, J1 to J2, J2 to J4, R1 to R3, R2 to R7
Connections:
- net BLK: now also C3.2, C5.2, C6.2, C7.2, C8.2, D3.2 (A), D4.2 (A), J5.1 (P1), J5.2 (P2), J8.2 (P2), R14.1, R16.1, R6.1, C1.2, C10.2, C11.2, C12.2, C13.2, C14.2, C15.2, C16.2, C9.2, D1.2 (A), D5.2 (A), D6.2 (A), D7.2 (A), D8.2 (A), J1.1 (P1), J1.2 (P2), J10.1 (P1), J10.2 (P2), J11.2 (P2), J12.2 (P2), J13.1 (P1), J13.2 (P2), J14.1 (P1), J14.2 (P2), J15.2 (P2), J16.2 (P2), J3.2 (P2), J6.1 (P1), J6.2 (P2), J7.2 (P2), J9.1 (P1), J9.2 (P2), R22.1, R24.1, R30.1, R32.1, U1.4 (V-), U1.4 (V-), U3.4 (V-), U3.4 (V-), U4.4 (V-), U4.4 (V-), U5.4 (V-), U5.4 (V-), U6.4 (V-), U6.4 (V-), U7.4 (V-), U7.4 (V-), U8.4 (V-), U8.4 (V-)
- net GND: no longer C3.2, C5.2, C6.2, C7.2, C8.2, D3.2 (A), D4.2 (A), J5.1 (P1), J5.2 (P2), J8.2 (P2), R12.2, R16.2
- net GRN: now also J8.4 (P4), J11.4 (P4), J12.4 (P4), J15.4 (P4), J16.4 (P4), J3.4 (P4), J7.4 (P4), U1.3 (+), U3.3 (+), U4.3 (+), U5.3 (+), U6.3 (+), U7.3 (+), U8.3 (+)
- net RED: now also C3.1, C7.1, C8.1, J5.3 (P3), J8.1 (P1), C11.1, C12.1, C15.1, C16.1, J1.3 (P3), J10.3 (P3), J11.1 (P1), J12.1 (P1), J13.3 (P3), J14.3 (P3), J15.1 (P1), J16.1 (P1), J3.1 (P1), J6.3 (P3), J7.1 (P1), J9.3 (P3), U1.8 (V+), U1.8 (V+), U3.8 (V+), U3.8 (V+), U4.8 (V+), U4.8 (V+), U5.8 (V+), U5.8 (V+), U6.8 (V+), U6.8 (V+), U7.8 (V+), U7.8 (V+), U8.8 (V+), U8.8 (V+)
- net Vout: now also C5.1, C6.1, D3.1 (K), D4.1 (K), J5.4 (P4), R10.2, R12.2, R13.1, R15.1, R5.1, C1.1, C10.1, C13.1, C14.1, C9.1, D1.1 (K), D5.1 (K), D6.1 (K), D7.1 (K), D8.1 (K), J1.4 (P4), J10.4 (P4), J13.4 (P4), J14.4 (P4), J6.4 (P4), J9.4 (P4), R18.2, R2.2, R20.2, R21.1, R23.1, R26.2, R28.2, R29.1, R31.1, U1.7, U3.7, U4.7, U5.7, U6.7, U7.7, U8.7
- net WHT: now also J8.3 (P3), J11.3 (P3), J12.3 (P3), J15.3 (P3), J16.3 (P3), J3.3 (P3), J7.3 (P3), U1.5 (+), U3.5 (+), U4.5 (+), U5.5 (+), U6.5 (+), U7.5 (+), U8.5 (+)
- net at R5.2: now also R1.1, U1.2 (-); no longer R6.1
- net at R6.2: now also R2.1, U1.6 (-)
- net at R11.2: now also U4.1; no longer R9.1
- net at R9.2: now also U3.1; no longer R10.1
- net at R15.2: now also R11.1, U4.2 (-); no longer R13.1
- net at R13.2: now also R9.1, U3.2 (-); no longer R14.1
- net at R14.2: now also R10.1, U3.6 (-); no longer J8.4 (P4)
- new net: R1.2, U1.1
- new net: R12.1, R16.2, U4.6 (-)
- new net: R19.1, R23.2, U6.2 (-)
- new net: R19.2, U6.1
- new net: R20.1, R24.2, U6.6 (-)
- new net: R17.1, R21.2, U5.2 (-)
- new net: R17.2, U5.1
- new net: R18.1, R22.2, U5.6 (-)
- new net: R27.1, R31.2, U8.2 (-)
- new net: R27.2, U8.1
- new net: R28.1, R32.2, U8.6 (-)
- new net: R25.1, R29.2, U7.2 (-)
- new net: R25.2, U7.1
- new net: R26.1, R30.2, U7.6 (-)
Other:
- moved on the sheet: C2, C4, D2, FID1, FID2, FID3, J2, J4, R3, R4, R7, R8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

Commit message: Checkpoint - first unit laid out
Parts:
- R14, R16, R22, R24, R30, R32, R6, R8: value 270K -> 390K
Connections:
- net BLK: no longer C10.2, C11.2, C12.2, C13.2, C14.2, C15.2, C16.2, C2.2, C4.2, C5.2, C6.2, C7.2, C8.2, C9.2, D2.2 (A), D3.2 (A), D4.2 (A), D5.2 (A), D6.2 (A), D7.2 (A), D8.2 (A), J10.1 (P1), J10.2 (P2), J11.2 (P2), J12.2 (P2), J13.1 (P1), J13.2 (P2), J14.1 (P1), J14.2 (P2), J15.2 (P2), J16.2 (P2), J2.1 (P1), J2.2 (P2), J4.2 (P2), J5.1 (P1), J5.2 (P2), J6.1 (P1), J6.2 (P2), J7.2 (P2), J8.2 (P2), J9.1 (P1), J9.2 (P2), R14.1, R16.1, R22.1, R24.1, R30.1, R32.1, R8.1, U2.4 (V-), U2.4 (V-), U3.4 (V-), U3.4 (V-), U4.4 (V-), U4.4 (V-), U5.4 (V-), U5.4 (V-), U6.4 (V-), U6.4 (V-), U7.4 (V-), U7.4 (V-), U8.4 (V-), U8.4 (V-)
- net GRN: no longer J11.4 (P4), J12.4 (P4), J15.4 (P4), J16.4 (P4), J4.4 (P4), J7.4 (P4), J8.4 (P4), U2.3 (+), U3.3 (+), U4.3 (+), U5.3 (+), U6.3 (+), U7.3 (+), U8.3 (+)
- net RED: no longer C11.1, C12.1, C15.1, C16.1, C4.1, C7.1, C8.1, J10.3 (P3), J11.1 (P1), J12.1 (P1), J13.3 (P3), J14.3 (P3), J15.1 (P1), J16.1 (P1), J2.3 (P3), J4.1 (P1), J5.3 (P3), J6.3 (P3), J7.1 (P1), J8.1 (P1), J9.3 (P3), U2.8 (V+), U2.8 (V+), U3.8 (V+), U3.8 (V+), U4.8 (V+), U4.8 (V+), U5.8 (V+), U5.8 (V+), U6.8 (V+), U6.8 (V+), U7.8 (V+), U7.8 (V+), U8.8 (V+), U8.8 (V+)
- net Vout: no longer C10.1, C13.1, C14.1, C2.1, C5.1, C6.1, C9.1, D2.1 (K), D3.1 (K), D4.1 (K), D5.1 (K), D6.1 (K), D7.1 (K), D8.1 (K), J10.4 (P4), J13.4 (P4), J14.4 (P4), J2.4 (P4), J5.4 (P4), J6.4 (P4), J9.4 (P4), R10.2, R12.2, R13.1, R15.1, R18.2, R20.2, R21.1, R23.1, R26.2, R28.2, R29.1, R31.1, R4.2, R7.1, U2.7, U3.7, U4.7, U5.7, U6.7, U7.7, U8.7
- net WHT: no longer J11.3 (P3), J12.3 (P3), J15.3 (P3), J16.3 (P3), J4.3 (P3), J7.3 (P3), J8.3 (P3), U2.5 (+), U3.5 (+), U4.5 (+), U5.5 (+), U6.5 (+), U7.5 (+), U8.5 (+)
- new net: C4.1, J2.3 (P3), J4.1 (P1), U2.8 (V+), U2.8 (V+)
- new net: C2.2, C4.2, D2.2 (A), J2.1 (P1), J2.2 (P2), J4.2 (P2), R8.1, U2.4 (V-), U2.4 (V-)
- new net: C2.1, D2.1 (K), J2.4 (P4), R4.2, R7.1, U2.7
- new net: J4.3 (P3), U2.5 (+)
- new net: J4.4 (P4), U2.3 (+)
- new net: C8.1, J6.3 (P3), J8.1 (P1), U4.8 (V+), U4.8 (V+)
- new net: C6.2, C8.2, D4.2 (A), J6.1 (P1), J6.2 (P2), J8.2 (P2), R16.1, U4.4 (V-), U4.4 (V-)
- new net: C6.1, D4.1 (K), J6.4 (P4), R12.2, R15.1, U4.7
- new net: J8.3 (P3), U4.5 (+)
- new net: J8.4 (P4), U4.3 (+)
- new net: C7.1, J5.3 (P3), J7.1 (P1), U3.8 (V+), U3.8 (V+)
- new net: C5.2, C7.2, D3.2 (A), J5.1 (P1), J5.2 (P2), J7.2 (P2), R14.1, U3.4 (V-), U3.4 (V-)
- new net: C5.1, D3.1 (K), J5.4 (P4), R10.2, R13.1, U3.7
- new net: J7.3 (P3), U3.5 (+)
- new net: J7.4 (P4), U3.3 (+)
- new net: C12.1, J10.3 (P3), J12.1 (P1), U6.8 (V+), U6.8 (V+)
- new net: C10.2, C12.2, D6.2 (A), J10.1 (P1), J10.2 (P2), J12.2 (P2), R24.1, U6.4 (V-), U6.4 (V-)
- new net: C10.1, D6.1 (K), J10.4 (P4), R20.2, R23.1, U6.7
- new net: J12.3 (P3), U6.5 (+)
- new net: J12.4 (P4), U6.3 (+)
- new net: C11.1, J11.1 (P1), J9.3 (P3), U5.8 (V+), U5.8 (V+)
- new net: C11.2, C9.2, D5.2 (A), J11.2 (P2), J9.1 (P1), J9.2 (P2), R22.1, U5.4 (V-), U5.4 (V-)
- new net: C9.1, D5.1 (K), J9.4 (P4), R18.2, R21.1, U5.7
- new net: J11.3 (P3), U5.5 (+)
- new net: J11.4 (P4), U5.3 (+)
- new net: C16.1, J14.3 (P3), J16.1 (P1), U8.8 (V+), U8.8 (V+)
- new net: C14.2, C16.2, D8.2 (A), J14.1 (P1), J14.2 (P2), J16.2 (P2), R32.1, U8.4 (V-), U8.4 (V-)
- new net: C14.1, D8.1 (K), J14.4 (P4), R28.2, R31.1, U8.7
- new net: J16.3 (P3), U8.5 (+)
- new net: J16.4 (P4), U8.3 (+)
- new net: C15.1, J13.3 (P3), J15.1 (P1), U7.8 (V+), U7.8 (V+)
- new net: C13.2, C15.2, D7.2 (A), J13.1 (P1), J13.2 (P2), J15.2 (P2), R30.1, U7.4 (V-), U7.4 (V-)
- new net: C13.1, D7.1 (K), J13.4 (P4), R26.2, R29.1, U7.7
- new net: J15.3 (P3), U7.5 (+)
- new net: J15.4 (P4), U7.3 (+)
Changed lines of the file:
@@
 	1    0    0    -1
 $EndComp
-Text Label 7800 950  0    40   ~ 0
-Vcc
-Text Label 8500 950  0    40   ~ 0
-Vout
 $Comp
 L 0.100_1X4 J4
@@
 	0    -1   1    0
 $EndComp
-Text Label 5450 1350 3    40   ~ 0
-RED
-Text Label 5550 1350 3    40   ~ 0
-BLK
-Text Label 5750 1350 3    40   ~ 0
-GRN
-Text Label 5850 1500 0    40   ~ 0
-WHT
 Wire Wire Line
 	5050 950  5050 1700
@@
 P 7950 1950
 F 0 "R8" V 8030 1950 50  0000 C CNN
-F 1 "270K" V 7950 1950 50  0000 C CNN
+F 1 "390K" V 7950 1950 50  0000 C CNN
 F 2 "_Passive:R_0603" V 7880 1950 50  0001 C CNN
 F 3 "" H 7950 1950 50  0000 C CNN
@@
 P 3850 1950
 F 0 "R6" V 3930 1950 50  0000 C CNN
-F 1 "270K" V 3850 1950 50  0000 C CNN
+F 1 "390K" V 3850 1950 50  0000 C CNN
 F 2 "_Passive:R_0603" V 3780 1950 50  0001 C CNN
 F 3 "" H 3850 1950 50  0000 C CNN
@@
 	1    0    0    -1
 $EndComp
-Text Label 7750 2550 0    40   ~ 0
-Vcc
-Text Label 8450 2550 0    40   ~ 0
-Vout
 $Comp
 L 0.100_1X4 J8
@@
 	0    -1   1    0
 $EndComp
-Text Label 5400 2950 3    40   ~ 0
-RED
-Text Label 5500 2950 3    40   ~ 0
-BLK
-Text Label 5700 2950 3    40   ~ 0
-GRN
-Text Label 5800 3100 0    40   ~ 0
-WHT
 Wire Wire Line
 	5000 2550 5000 3300
@@
 P 7900 3550
 F 0 "R16" V 7980 3550 50  0000 C CNN
-F 1 "270K" V 7900 3550 50  0000 C CNN
+F 1 "390K" V 7900 3550 50  0000 C CNN
 F 2 "_Passive:R_0603" V 7830 3550 50  0001 C CNN
 F 3 "" H 7900 3550 50  0000 C CNN
@@
 	1    0    0    -1
 $EndComp
-Text Label 3650 2550 0    40   ~ 0
-Vcc
-Text Label 4350 2550 0    40   ~ 0
-Vout
 $Comp
 L 0.100_1X4 J7
@@
 	0    -1   1    0
 $EndComp
-Text Label 1300 2950 3    40   ~ 0
-RED
-Text Label 1400 2950 3    40   ~ 0
-BLK
-Text Label 1600 2950 3    40   ~ 0
-GRN
-Text Label 1700 3100 0    40   ~ 0
-WHT
 Wire Wire Line
 	900  2550 900  3300
@@
 P 3800 3550
 F 0 "R14" V 3880 3550 50  0000 C CNN
-F 1 "270K" V 3800 3550 50  0000 C CNN
+F 1 "390K" V 3800 3550 50  0000 C CNN
 F 2 "_Passive:R_0603" V 3730 3550 50  0001 C CNN
 F 3 "" H 3800 3550 50  0000 C CNN
@@
 	1    0    0    -1
 $EndComp
-Text Label 7750 4150 0    40   ~ 0
-Vcc
-Text Label 8450 4150 0    40   ~ 0
-Vout
 $Comp
 L 0.100_1X4 J12
@@
 	0    -1   1    0
 $EndComp
-Text Label 5400 4550 3    40   ~ 0
-RED
-Text Label 5500 4550 3    40   ~ 0
-BLK
-Text Label 5700 4550 3    40   ~ 0
-GRN
-Text Label 5800 4700 0    40   ~ 0
-WHT
 Wire Wire Line
 	5000 4150 5000 4900
@@
 P 7900 5150
 F 0 "R24" V 7980 5150 50  0000 C CNN
-F 1 "270K" V 7900 5150 50  0000 C CNN
+F 1 "390K" V 7900 5150 50  0000 C CNN
 F 2 "_Passive:R_0603" V 7830 5150 50  0001 C CNN
 F 3 "" H 7900 5150 50  0000 C CNN
@@
 	1    0    0    -1
 $EndComp
-Text Label 3650 4150 0    40   ~ 0
-Vcc
-Text Label 4350 4150 0    40   ~ 0
-Vout
 $Comp
 L 0.100_1X4 J11
@@
 	0    -1   1    0
 $EndComp
-Text Label 1300 4550 3    40   ~ 0
-RED
-Text Label 1400 4550 3    40   ~ 0
-BLK
-Text Label 1600 4550 3    40   ~ 0
-GRN
-Text Label 1700 4700 0    40   ~ 0
-WHT
 Wire Wire Line
 	900  4150 900  4900
@@
 P 3800 5150
 F 0 "R22" V 3880 5150 50  0000 C CNN
-F 1 "270K" V 3800 5150 50  0000 C CNN
+F 1 "390K" V 3800 5150 50  0000 C CNN
 F 2 "_Passive:R_0603" V 3730 5150 50  0001 C CNN
 F 3 "" H 3800 5150 50  0000 C CNN
@@
 	1    0    0    -1
 $EndComp
-Text Label 7700 5750 0    40   ~ 0
-Vcc
-Text Label 8400 5750 0    40   ~ 0
-Vout
 $Comp
 L 0.100_1X4 J16
@@
 	0    -1   1    0
 $EndComp
-Text Label 5350 6150 3    40   ~ 0
-RED
-Text Label 5450 6150 3    40   ~ 0
-BLK
-Text Label 5650 6150 3    40   ~ 0
-GRN
-Text Label 5750 6300 0    40   ~ 0
-WHT
 Wire Wire Line
 	4950 5750 4950 6500
@@
 P 7850 6750
 F 0 "R32" V 7930 6750 50  0000 C CNN
-F 1 "270K" V 7850 6750 50  0000 C CNN
+F 1 "390K" V 7850 6750 50  0000 C CNN
 F 2 "_Passive:R_0603" V 7780 6750 50  0001 C CNN
 F 3 "" H 7850 6750 50  0000 C CNN
@@
 	1    0    0    -1
 $EndComp
-Text Label 3600 5750 0    40   ~ 0
-Vcc
-Text Label 4300 5750 0    40   ~ 0
-Vout
 $Comp
 L 0.100_1X4 J15
@@
 	0    -1   1    0
 $EndComp
-Text Label 1250 6150 3    40   ~ 0
-RED
-Text Label 1350 6150 3    40   ~ 0
-BLK
-Text Label 1550 6150 3    40   ~ 0
-GRN
-Text Label 1650 6300 0    40   ~ 0
-WHT
 Wire Wire Line
 	850  5750 850  6500
@@
 P 3750 6750
 F 0 "R30" V 3830 6750 50  0000 C CNN
-F 1 "270K" V 3750 6750 50  0000 C CNN
+F 1 "390K" V 3750 6750 50  0000 C CNN
 F 2 "_Passive:R_0603" V 3680 6750 50  0001 C CNN
 F 3 "" H 3750 6750 50  0000 C CNN
